Commit message: added joint limits

File: rrbot_description/urdf/rrbot.xacro (robot description, xacro)
@@ -45,9 +45,10 @@
     </inertial>
   </link>
-  <joint name="joint1" type="continuous">
+  <joint name="joint1" type="revolute">
     <parent link="link1"/>
     <child link="link2"/>
     <origin xyz="0 ${width} ${height1 - axel_offset}" rpy="0 0 0"/>
     <axis xyz="0 1 0"/>
+    <limit effort="30" velocity="1.0" lower="-2" upper="2" />
     <dynamics damping="0.7"/>
   </joint>
@@ -76,9 +77,10 @@
     </inertial>
   </link>
-  <joint name="joint2" type="continuous">
+  <joint name="joint2" type="revolute">
     <parent link="link2"/>
     <child link="link3"/>
     <origin xyz="0 ${width} ${height2 - axel_offset*2}" rpy="0 0 0"/>
     <axis xyz="0 1 0"/>
+    <limit effort="30" velocity="1.0" lower="-2" upper="2" />
     <dynamics damping="0.7"/>
   </joint>
